Commit message: Sim customization, rope control

File: isaaclab/RopeUntyingRobot/assets/rope_chain.urdf (robot description, URDF)
Before this commit: robot rope_chain, 31 links, 30 joints
Joints:
- joint rope_pitch_0: limit lower=-0.523599 upper=0.523599 effort=0.1 velocity=10.0 -> lower=-2.094395 upper=2.094395 effort=0.1 velocity=10.0
- joint rope_pitch_1: limit lower=-0.523599 upper=0.523599 effort=0.1 velocity=10.0 -> lower=-2.094395 upper=2.094395 effort=0.1 velocity=10.0
- joint rope_pitch_10: limit lower=-0.523599 upper=0.523599 effort=0.1 velocity=10.0 -> lower=-2.094395 upper=2.094395 effort=0.1 velocity=10.0
- joint rope_pitch_11: limit lower=-0.523599 upper=0.523599 effort=0.1 velocity=10.0 -> lower=-2.094395 upper=2.094395 effort=0.1 velocity=10.0
- joint rope_pitch_12: limit lower=-0.523599 upper=0.523599 effort=0.1 velocity=10.0 -> lower=-2.094395 upper=2.094395 effort=0.1 velocity=10.0
- joint rope_pitch_13: limit lower=-0.523599 upper=0.523599 effort=0.1 velocity=10.0 -> lower=-2.094395 upper=2.094395 effort=0.1 velocity=10.0
- joint rope_pitch_14: limit lower=-0.523599 upper=0.523599 effort=0.1 velocity=10.0 -> lower=-2.094395 upper=2.094395 effort=0.1 velocity=10.0
- joint rope_pitch_2: limit lower=-0.523599 upper=0.523599 effort=0.1 velocity=10.0 -> lower=-2.094395 upper=2.094395 effort=0.1 velocity=10.0
- joint rope_pitch_3: limit lower=-0.523599 upper=0.523599 effort=0.1 velocity=10.0 -> lower=-2.094395 upper=2.094395 effort=0.1 velocity=10.0
- joint rope_pitch_4: limit lower=-0.523599 upper=0.523599 effort=0.1 velocity=10.0 -> lower=-2.094395 upper=2.094395 effort=0.1 velocity=10.0
- joint rope_pitch_5: limit lower=-0.523599 upper=0.523599 effort=0.1 velocity=10.0 -> lower=-2.094395 upper=2.094395 effort=0.1 velocity=10.0
- joint rope_pitch_6: limit lower=-0.523599 upper=0.523599 effort=0.1 velocity=10.0 -> lower=-2.094395 upper=2.094395 effort=0.1 velocity=10.0
- joint rope_pitch_7: limit lower=-0.523599 upper=0.523599 effort=0.1 velocity=10.0 -> lower=-2.094395 upper=2.094395 effort=0.1 velocity=10.0
- joint rope_pitch_8: limit lower=-0.523599 upper=0.523599 effort=0.1 velocity=10.0 -> lower=-2.094395 upper=2.094395 effort=0.1 velocity=10.0
- joint rope_pitch_9: limit lower=-0.523599 upper=0.523599 effort=0.1 velocity=10.0 -> lower=-2.094395 upper=2.094395 effort=0.1 velocity=10.0
- joint rope_yaw_0: limit lower=-0.523599 upper=0.523599 effort=0.1 velocity=10.0 -> lower=-2.094395 upper=2.094395 effort=0.1 velocity=10.0
- joint rope_yaw_1: limit lower=-0.523599 upper=0.523599 effort=0.1 velocity=10.0 -> lower=-2.094395 upper=2.094395 effort=0.1 velocity=10.0
- joint rope_yaw_10: limit lower=-0.523599 upper=0.523599 effort=0.1 velocity=10.0 -> lower=-2.094395 upper=2.094395 effort=0.1 velocity=10.0
- joint rope_yaw_11: limit lower=-0.523599 upper=0.523599 effort=0.1 velocity=10.0 -> lower=-2.094395 upper=2.094395 effort=0.1 velocity=10.0
- joint rope_yaw_12: limit lower=-0.523599 upper=0.523599 effort=0.1 velocity=10.0 -> lower=-2.094395 upper=2.094395 effort=0.1 velocity=10.0
- joint rope_yaw_13: limit lower=-0.523599 upper=0.523599 effort=0.1 velocity=10.0 -> lower=-2.094395 upper=2.094395 effort=0.1 velocity=10.0
- joint rope_yaw_14: limit lower=-0.523599 upper=0.523599 effort=0.1 velocity=10.0 -> lower=-2.094395 upper=2.094395 effort=0.1 velocity=10.0
- joint rope_yaw_2: limit lower=-0.523599 upper=0.523599 effort=0.1 velocity=10.0 -> lower=-2.094395 upper=2.094395 effort=0.1 velocity=10.0
- joint rope_yaw_3: limit lower=-0.523599 upper=0.523599 effort=0.1 velocity=10.0 -> lower=-2.094395 upper=2.094395 effort=0.1 velocity=10.0
- joint rope_yaw_4: limit lower=-0.523599 upper=0.523599 effort=0.1 velocity=10.0 -> lower=-2.094395 upper=2.094395 effort=0.1 velocity=10.0
- joint rope_yaw_5: limit lower=-0.523599 upper=0.523599 effort=0.1 velocity=10.0 -> lower=-2.094395 upper=2.094395 effort=0.1 velocity=10.0
- joint rope_yaw_6: limit lower=-0.523599 upper=0.523599 effort=0.1 velocity=10.0 -> lower=-2.094395 upper=2.094395 effort=0.1 velocity=10.0
- joint rope_yaw_7: limit lower=-0.523599 upper=0.523599 effort=0.1 velocity=10.0 -> lower=-2.094395 upper=2.094395 effort=0.1 velocity=10.0
- joint rope_yaw_8: limit lower=-0.523599 upper=0.523599 effort=0.1 velocity=10.0 -> lower=-2.094395 upper=2.094395 effort=0.1 velocity=10.0
- joint rope_yaw_9: limit lower=-0.523599 upper=0.523599 effort=0.1 velocity=10.0 -> lower=-2.094395 upper=2.094395 effort=0.1 velocity=10.0
